File: Vega_EV1/OtterX.kicad_pcb (KiCad board)
At the start: 4 copper layers, 170.1 x 170.1 mm, 180 parts, among them J1 VERA_CONN, J10 1.5MB RAM Expansion, J11 KMDGX-6SG, J12 VIA1 Extra Pins, J14 Flash WR EN, J16 ATX-24, J17 SNES23, J18 SNES0, J19 SNES1, J2 VIA2 Header, J21 ISP, J25 PS2 Pwr Src, J26 Front Panel, J27 EXTRAM_ENABLE, J29 AudioPlug3, J3 IEC, J5 YM CT Out, J6 Ext. NMI, J7 RTC GPIO, J9 I2C, K1 HK19F, P1 60 Pin Edge Conn, Q1 2N7000, Q2 2N7000, Q3 2N7000, SW1 FSM4JH, SW2 FSM4JH, SW3 FSM4JH, U1 W65C02S, U11 74ACT163, U12 ATtiny861-20P, U13 MCP7940N-xP, U14 74AHCT00, U15 74AHCT02, U16 74AHCT04, U17 74AHCT02, U18 74AHCT32, U19 74AHCT20, U2 W65C22S, U20 74AHCT20, U21 74AHCT138, U22 TL074, U24 YM2151, U25 YM3012, U26 LM324, U4 74AHCT10, U5 74AHCT273, U6 74AHCT273, U7 SST39SF040, U8 AS6C1008-55PCN, U9 AS6C4008-55PCN, X1 ACH-16.000MHZ-EK, X2 ECS-2100AX-3.579545MHZ, Y1 ECS-.327-6-13X

Commit message: Misc layout fixes.
Parts:
- J12: footprint Connector_PinHeader_2.54mm:PinHeader_2x04_P2.54mm_Vertical -> Connector_PinSocket_2.54mm:PinSocket_2x04_P2.54mm_Horizontal
- J17: footprint Connector_PinSocket_2.54mm:PinSocket_2x03_P2.54mm_Vertical -> Connector_PinSocket_2.54mm:PinSocket_2x03_P2.54mm_Horizontal
- moved C14 68.4 mm to (148.6, 38.2), turned to 90 degrees
- moved C13 58.8 mm to (146.1, 38.2), turned to 90 degrees
- moved J12 42.1 mm to (168.6, 24.8), turned to -90 degrees
- moved C20 18.8 mm to (145.9, 24.6), turned to 90 degrees
- moved C19 11.4 mm to (148.4, 25.1)
- moved J17 11.0 mm to (156.5, 24.9)
- moved R12 1.60 mm to (154.6, 31.8)
- moved R10 1.45 mm to (151.4, 31.8)
- moved J5 0.90 mm to (44.6, 69.2)
- moved J27 0.50 mm to (31.1, 134.3)
- moved K1 0.09 mm to (53.0, 33.9)
Connections:
- J12 pad 1: +5V -> V1PB2
- J12 pad 2: CA1 -> GND
- J12 pad 3: V1PB0 -> V1PB1
- J12 pad 4: CA2 -> CB2
- J12 pad 5: V1PB1 -> V1PB0
- J12 pad 6: CB2 -> CA2
- J12 pad 7: V1PB2 -> +5V
- J12 pad 8: GND -> CA1
Routing:
- net +5V: track 1490.8 -> 1401.3 mm, vias 30 -> 28
- net CA2: track 17.2 -> 55.1 mm
- net ~{PG2A}: track 97.0 -> 61.3 mm
- net CA1: track 13.0 -> 41.4 mm, vias 1 -> 2
- net NESDAT3: track 39.2 -> 27.3 mm, vias 1 -> 0
- net NESLATCH: track 108.1 -> 96.6 mm, vias 2 -> 0
- net NESCLK: track 101.8 -> 91.1 mm, vias 3 -> 1
- net NESDAT2: track 33.4 -> 26.8 mm
- net V1PB0: track 53.9 -> 47.3 mm
- net CB2: track 78.7 -> 84.7 mm
- net IECATTO: track 71.3 -> 73.7 mm
- net NESDAT0: track 25.6 -> 24.1 mm
- net SDA: track 369.1 -> 370.2 mm
- net SCL: track 382.3 -> 383.3 mm
- net /SMC/RESBTN_PD: track 162.7 -> 161.8 mm
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Other:
- board text added: "CA1"
- board text added: "CA2"
- board text added: "CB2"
- board text added: "CLK"
- board text added: "DAT2"
- board text added: "DAT3"
- board text added: "LATCH"
- board text added: "PB0"
- board text added: "PB1"
- board text added: "PB2"
- board text added: "YM CT1/2"
