File: Vega_EV1/OtterX.kicad_pcb (KiCad board)
At the start: 4 copper layers, 170.1 x 170.1 mm, 187 parts, among them J1 VERA_CONN, J10 1.5MB RAM Expansion, J11 KMDGX-6SG, J12 VIA1 Extra Pins, J14 Flash WR EN, J16 ATX-24, J17 IDC_2x03, J18 SNES0, J19 SNES1, J2 VIA2 Header, J21 IDC_2x03, J25 PS2 Pwr Src, J26 Front Panel, J27 EXTRAM_ENABLE, J29 AudioPlug3, J3 IDC_2x03, J5 YM CT Out, J6 Ext. NMI, J7 RTC GPIO, J9 I2C, K1 HK19F, P1 60 Pin Edge Conn, Q1 2N7000, Q2 2N7000, Q3 2N7000, SW1 FSM4JH, SW2 FSM4JH, SW3 FSM4JH, U1 W65C816S, U11 74ACT163, U12 ATtiny861-20P, U13 MCP7940N-xP, U14 74ACT00, U15 74AHCT02, U16 74AHCT04, U17 74AHCT02, U18 74AHCT32, U19 74AC20, U2 W65C22S, U20 74AC20, U21 74AHCT138, U22 TL074, U24 YM2151, U25 YM3012, U26 LM324, U3 74LS06, U4 74AC10, U5 74AHCT273, U6 74AHCT273, U7 SST39SF040, U8 AS6C1008-55PCN, U9 AS6C4008-55PCN, X1 ACH-16.000MHZ-EK, X2 ECS-2100AX-3.579545MHZ, Y1 ECS-.327-6-13X

Commit message: Vega production Gerber Out
Routing:
- net SCL: track 385.7 -> 384.5 mm
- net Net-(JP3-A): track 143.2 -> 142.5 mm
- net GND: vias 88 -> 157
Other:
- board text added: "SNES1"
- board text added: "SNES2"
