File: Vega_EV1/audio.kicad_sch (KiCad schematic)
At the start: 22 parts, among them J5 YM CT Out, K1 HK19F, Q3 2N7000, U24 YM2151, U25 YM3012, U26 LM324, X2 ECS-2100AX-3.579545MHZ

Commit message: Fix #16, widen transistor footprints
Parts:
- Q3: footprint Package_TO_SOT_THT:TO-92_Inline -> Package_TO_SOT_THT:TO-92_Inline_Wide
Changed lines of the file:
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@@
 			)
 		)
-		(property "Footprint" "Package_TO_SOT_THT:TO-92_Inline"
+		(property "Footprint" "Package_TO_SOT_THT:TO-92_Inline_Wide"
 			(at 206.375 146.685 0)
 			(effects

Commit message: More space between Edge and YM2151 Add IEC logic back in IDC headers for NES and IEC
Parts:
- D19: footprint Diode_THT:D_DO-35_SOD27_P7.62mm_Horizontal -> Diode_THT:D_DO-34_SOD68_P7.62mm_Horizontal
Changed lines of the file:
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@@
 	(label "D6"
 		(at 73.66 86.36 0)
-		(fields_autoplaced yes)
 		(effects
 			(font
@@
 	(label "YMVREF_IN"
 		(at 187.833 55.245 0)
-		(fields_autoplaced yes)
 		(effects
 			(font
@@
 	(label "D1"
 		(at 73.66 73.66 0)
-		(fields_autoplaced yes)
 		(effects
 			(font
@@
 	(label "~{RES}"
 		(at 189.865 135.255 0)
-		(fields_autoplaced yes)
 		(effects
 			(font
@@
 	(label "YMSAMP_OUT"
 		(at 187.96 59.817 0)
-		(fields_autoplaced yes)
 		(effects
 			(font
@@
 	(label "YM_CT1"
 		(at 59.69 96.52 0)
-		(fields_autoplaced yes)
 		(effects
 			(font
@@
 	(label "YMANL_5V"
 		(at 167.64 33.02 0)
-		(fields_autoplaced yes)
 		(effects
 			(font
@@
 	(label "D7"
 		(at 73.66 88.9 0)
-		(fields_autoplaced yes)
 		(effects
 			(font
@@
 	(label "YM_COM"
 		(at 187.325 64.897 0)
-		(fields_autoplaced yes)
 		(effects
 			(font
@@
 	(label "D2"
 		(at 73.66 76.2 0)
-		(fields_autoplaced yes)
 		(effects
 			(font
@@
 	(label "D5"
 		(at 73.66 83.82 0)
-		(fields_autoplaced yes)
 		(effects
 			(font
@@
 	(label "SO"
 		(at 137.16 59.69 0)
-		(fields_autoplaced yes)
 		(effects
 			(font
@@
 	(label "YMVREF_OUT"
 		(at 187.071 50.927 0)
-		(fields_autoplaced yes)
 		(effects
 			(font
@@
 	(label "YM_CT2"
 		(at 58.42 93.98 0)
-		(fields_autoplaced yes)
 		(effects
 			(font
@@
 	(label "SH1"
 		(at 135.89 64.77 0)
-		(fields_autoplaced yes)
 		(effects
 			(font
@@
 	(label "D3"
 		(at 73.66 78.74 0)
-		(fields_autoplaced yes)
 		(effects
 			(font
@@
 	(label "YMANL_CH1"
 		(at 187.325 92.075 0)
-		(fields_autoplaced yes)
 		(effects
 			(font
@@
 	(label "YMVREF_BIAS"
 		(at 186.055 45.72 0)
-		(fields_autoplaced yes)
 		(effects
 			(font
@@
 	(label "SH2"
 		(at 135.89 67.31 0)
-		(fields_autoplaced yes)
 		(effects
 			(font
@@
 	(label "YM_CLK"
 		(at 73.66 49.53 0)
-		(fields_autoplaced yes)
 		(effects
 			(font
@@
 	(label "YMANL_CH2"
 		(at 189.865 73.66 0)
-		(fields_autoplaced yes)
 		(effects
 			(font
@@
 	(label "YM_CLK2"
 		(at 137.16 54.61 0)
-		(fields_autoplaced yes)
 		(effects
 			(font
@@
 	(label "D4"
 		(at 73.66 81.28 0)
-		(fields_autoplaced yes)
 		(effects
 			(font
@@
 	(label "D0"
 		(at 73.66 71.12 0)
-		(fields_autoplaced yes)
 		(effects
 			(font
@@
 			)
 		)
-		(property "Footprint" "Diode_THT:D_DO-35_SOD27_P7.62mm_Horizontal"
+		(property "Footprint" "Diode_THT:D_DO-34_SOD68_P7.62mm_Horizontal"
 			(at 240.03 116.84 0)
 			(effects
