File: Vega_EV1/Audio_Mixer.kicad_sch (KiCad schematic)
At the start: 17 parts, among them U22 TL074

Commit message: Change 2.2u cap footprint; update MemoryExpansion
Parts:
- C46, C47: footprint Capacitor_THT:C_Rect_L10.3mm_W5.7mm_P7.50mm_MKS4 -> Capacitor_THT:C_Rect_L7.2mm_W5.5mm_P5.00mm_FKS2_FKP2_MKS2_MKP2; MPN (none) -> MKS2B042201F00JSSD
Changed lines of the file:
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@@
 			)
 		)
-		(property "Footprint" "Capacitor_THT:C_Rect_L10.3mm_W5.7mm_P7.50mm_MKS4"
+		(property "Footprint" "Capacitor_THT:C_Rect_L7.2mm_W5.5mm_P5.00mm_FKS2_FKP2_MKS2_MKP2"
 			(at 128.905 61.595 0)
 			(effects
@@
 		(property "Description" ""
 			(at 128.905 61.595 0)
+			(effects
+				(font
+					(size 1.27 1.27)
+				)
+				(hide yes)
+			)
+		)
+		(property "MPN" "MKS2B042201F00JSSD"
+			(at 128.905 61.595 90)
 			(effects
 				(font
@@
 			)
 		)
-		(property "Footprint" "Capacitor_THT:C_Rect_L10.3mm_W5.7mm_P7.50mm_MKS4"
+		(property "Footprint" "Capacitor_THT:C_Rect_L7.2mm_W5.5mm_P5.00mm_FKS2_FKP2_MKS2_MKP2"
 			(at 125.73 159.385 0)
 			(effects
@@
 			)
 		)
-		(pin "1"
-		)
-		(pin "2"
-		)
-		(instances
-			(project "OtterX"
-				(path "/e63e39d7-6ac0-4ffd-8aa3-1841a4541b55/35c1273b-9984-4872-b2ba-d9345784fd1c/e50dd233-8666-4e51-adc9-17748422bd2a"
+		(property "MPN" "MKS2B042201F00JSSD"
+			(at 125.73 159.385 90)
+			(effects
+				(font
+					(size 1.27 1.27)
+				)
+				(hide yes)
+			)
+		)
+		(pin "1"
+		)
+		(pin "2"
+		)
+		(instances
+			(project ""
+				(path "/e63e39d7-6ac0-4ffd-8aa3-1841a4541b55"
 					(reference "C47")
+					(unit 1)
+				)
+				(path "/e63e39d7-6ac0-4ffd-8aa3-1841a4541b55/35c1273b-9984-4872-b2ba-d9345784fd1c/e50dd233-8666-4e51-adc9-17748422bd2a"
+					(reference "C47")
