File: IEC_Dongle/IEC_Dongle.kicad_pcb (KiCad board)
At the start: 2 copper layers, 40 x 47 mm, 14 parts, among them J1 SDF-60J, J2 IDC_2x03

Commit message: Vega production Gerber Out
Other:
- board text added: "Rev: EV1"
Changed lines of the file:
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@@
+		)
+	)
+	(gr_text "Rev:\nEV1"
+		(at 164.15 69.15 0)
+		(layer "F.SilkS")
+		(effects
+			(font
+				(size 1 1)
+				(thickness 0.1)
+			)
+			(justify left bottom)
 		)
 	)
